Commit message: resolved friction prioblem, controller still broken

File: src/scenarios/models/ddmr/model.sdf.xacro (robot description, xacro)
@@ -136,4 +136,17 @@
             </cylinder>
           </geometry>
+          <surface>
+            <friction>
+              <ode>
+                <!-- high traction forward -->
+                <mu>1.0</mu>
+                <mu2>0.02</mu2>
+                <!-- wheel rolling direction -->
+                <fdir1>0 1 0</fdir1>
+                <slip1>0.0</slip1>
+                <slip2>0.4</slip2>
+              </ode>
+            </friction>
+          </surface>
         </collision>
         <xacro:cylinder_inertia m="0.5" r="${wheel_radius}" h="${wheel_width}"/>
@@ -146,7 +159,11 @@
           <xyz>0 1 0</xyz>
           <limit>
-            <lower>-inf</lower>
-            <upper>inf</upper>
+            <lower>-1e16</lower>
+            <upper>1e16</upper>
           </limit>
+          <dynamics>
+            <damping>0.05</damping>
+            <friction>0.0</friction>
+          </dynamics>
         </axis>
       </joint>
@@ -173,4 +190,12 @@
           </sphere>
         </geometry>
+        <surface>
+          <friction>
+            <ode>
+              <mu>0.01</mu>
+              <mu2>0.01</mu2>
+            </ode>
+          </friction>
+        </surface>
       </collision>
       <xacro:sphere_inertia m="0.5" r="${(wheel_radius+wheel_zoff-(base_height/2))}"/>
